Commit message: updated
this is the updated design of tricycle robot

File: tricycle.xacro (robot description, xacro)
@@ -9,5 +9,7 @@
 	         <cylinder length='3' radius='0.1'/>
 	        </geometry>
-			<material name="red" />
+			<material name="red" >
+			<color rgba="1.0 0.0 0.0 1.0 "/>
+			</material>
 	    </visual>
 </link>
@@ -41,18 +43,22 @@
 <link name="left_back_wheel">
 	    <visual>
-	    <origin xyz="1.5 0 0" rpy="0 1.5 0" />
+	    <origin xyz="0 0 0" rpy="0 1.5 0" />
 			<geometry>
 	         <cylinder length = "${wheel_length}" radius="${wheel_radius}"/>
 	        </geometry>
-			<material name="magenta" />
+			<material name="blue">
+			<color rgba="0.0 0.0 0.8 1.0 "/>
+			</material>
 	    </visual>
 </link>
 <link name="right_back_wheel">
 	    <visual>
-	    <origin xyz="-1.5 0 0" rpy="0 1.5 0" />
+	    <origin xyz="0 0 0" rpy="0 1.5 0" />
 			<geometry>
 	         <cylinder length = "${wheel_length}" radius="${wheel_radius}"/>
 	        </geometry>
-			<material name="magenta" />
+			<material name="blue">
+			<color rgba="0.0 0.0 0.8 1.0 "/>
+			</material>
 	    </visual>
 </link>
@@ -97,20 +103,35 @@
 <link name="front_wheel">
 	    <visual>
-	    <origin xyz="0 5 0" rpy="0 1.5 0" />
+	    <origin xyz="0 0 0" rpy="0 1.5 0" />
 			<geometry>
 	         <cylinder length = "${wheel_length}" radius="${wheel_radius}"/>
 	        </geometry>
-			<material name="magenta" />
+			<material name="blue" />
 	    </visual>
 </link>
 <link name="camera">
 	    <visual>
-			<origin xyz="0 3 2.5" rpy="0 0 0" />
+			<origin xyz="0 3 2.3" rpy="0 0 0" />
+			<geometry>
+	         <cylinder length = "0.3" radius="0.2"/>
+	        </geometry>
+			<material name="white">
+			<color rgba="1 1 1 1.0 "/>
+			</material>
+	    </visual>
+</link>
+<!--
+<link name="camera">
+	    <visual>
+			<origin xyz="0 3 2" rpy="0 0 0" />
 			<geometry>
 	         <box size='0.5 0.5 0.5'/>
 	        </geometry>
-			<material name="blue" />
-	    </visual>
-</link>
+			<material name="white">
+			<color rgba="1 1 1 1.0 "/>
+			</material>
+	    </visual>
+</link>
+-->
 <joint name="as_to_arm" type="fixed">
     <origin xyz="0 0 0" rpy="0 0 0"/>
@@ -131,15 +152,15 @@
  </joint>
  <joint name="bl_to_lbw" type="revolute">
-    <origin xyz="0 0 0" rpy="0 0 0"/>
+    <origin xyz="1.5 0 0" rpy="0 0 0" />
     <parent link="base_link"/>
     <child link="left_back_wheel"/>
-    <axis xyz = "0 0 1" />
+    <axis xyz = "1 0 0 " />
     <limit effort ="1000.0" lower="-1.0" upper="1.0" velocity="0.5"/>
  </joint>
  <joint name="bl_to_rbw" type="revolute">
-    <origin xyz="0 0 0" rpy="0 0 0"/>
+    <origin xyz="-1.5 0 0" rpy="0 0 0" />
     <parent link="base_link"/>
     <child link="right_back_wheel"/>
-    <axis xyz = "0 0 1" />
+    <axis xyz = "1 0 0" />
     <limit effort ="1000.0" lower="-1.0" upper="1.0" velocity="0.5"/>
  </joint>
@@ -167,8 +188,8 @@
  </joint>
  <joint name="ls_to_fw" type="revolute">
-    <origin xyz="0 0 0" rpy="0 0 0"/>
+    <origin xyz="0.2 4.5 0" rpy="0 0 0" />
     <parent link="lower_support"/>
     <child link="front_wheel"/>
-    <axis xyz = "0 0 1" />
+    <axis xyz = "1 0 0" />
     <limit effort ="1000.0" lower="-1.0" upper="1.0" velocity="0.5"/>
  </joint>
